File: pcb/FC/connectors.kicad_sch (KiCad schematic)
At the start: 16 parts, among them J1 FC-ESC, J2 MIC_1, J3 MIC_2, J4 SCREEN, J5 SERVO, J6 SPEAKER, J7 RC

Commit message: Add companion bring-up, base station features, and PCB updates
Document the verified hardware state and wire protocol, add companion display/audio/camera/telemetry drivers, expand the Python base station and tests, and capture PCB source/manufacturing changes. Stop tracking generated caches and local project state.
Parts:
- renumbered D3 to D?, D5 to D?, FPC1 to FPC?, H3 to H?, H1 to H?, H4 to H?, H2 to H?, J1 to J?, J4 to J?, J5 to J?, J7 to J?, J2 to J?, J3 to J?, J6 to J?, R21 to R?, R19 to R?
